Commit message: melhor identação do código e adição de lidar e suporte para camera

File: urdf/base.xacro (robot description, xacro)
@@ -3,5 +3,4 @@
   <xacro:include filename="$(find ros_commons)/urdf/domain.xacro"/>
   <xacro:property name="M" value="0.001"/>
-  <xacro:property name="DEG" value="0.01745329251"/>
   <xacro:property name="ground_clearance" value="${23 * M}"/>
   <xacro:property name="wheel_diameter" value="${84 * M}"/>
@@ -14,13 +13,25 @@
   <xacro:property name="body_height" value="${overall_height_base - ground_clearance}"/>
   <xacro:property name="body_z_offset" value="${ground_clearance + 0.5 * body_height}"/>
-  <!-- O eixo deve estar abaixo do centro do body, de forma que as rodas toquem o chão -->
-  <!-- O offset é negativo porque o eixo está abaixo do centro do body -->
   <xacro:property name="wheel_axle_z_offset" value="${wheel_radius - 0.5 * body_height - ground_clearance}"/>
-  <!-- wheel_separation: distância entre os centros das rodas esquerda e direita -->
   <xacro:property name="wheel_separation" value="${body_width - wheel_thickness}"/>
   <xacro:macro name="wheels" params="position">
-    <xacro:solid_cylinder name="wheel_${position}_left" length="${wheel_thickness}" radius="${wheel_radius}" roll="${90.0 * DEG}"/>
-    <xacro:solid_cylinder name="wheel_${position}_right" length="${wheel_thickness}" radius="${wheel_radius}" roll="${90.0 * DEG}"/>
-    <xacro:solid_cylinder name="wheel_${position}_axle" length="${wheel_separation}" radius="0.005" roll="${90.0 * DEG}"/>
+    <xacro:solid_cylinder
+      name="wheel_${position}_left"
+      length="${wheel_thickness}"
+      radius="${wheel_radius}"
+      roll="${90.0 * DEG}"
+    />
+    <xacro:solid_cylinder
+      name="wheel_${position}_right"
+      length="${wheel_thickness}"
+      radius="${wheel_radius}"
+      roll="${90.0 * DEG}"
+    />
+    <xacro:solid_cylinder
+      name="wheel_${position}_axle"
+      length="${wheel_separation}"
+      radius="0.005"
+      roll="${90.0 * DEG}"
+    />
     <xacro:joint_continuous
       name="joint_wheel_${position}_left"
@@ -28,5 +39,6 @@
       child="wheel_${position}_left"
       y="${(wheel_separation + wheel_thickness) * 0.5}"
-      axis="0 1 0"/>
+      axis="0 1 0"
+    />
     <xacro:joint_continuous
       name="joint_wheel_${position}_right"
@@ -34,8 +46,9 @@
       child="wheel_${position}_right"
       y="${(wheel_separation + wheel_thickness) * -0.5}"
-      axis="0 1 0"/>
+      axis="0 1 0"
+    />
   </xacro:macro>
-  <xacro:wheels position="front"/>
-  <xacro:wheels position="rear"/>
+  <!-- Link base para conectar o body -->
+  <link name="base_link"/>
   <!-- Corpo do robô -->
   <xacro:solid_block
@@ -44,9 +57,21 @@
     size_y="${body_width}"
     size_z="${body_height}"/>
+  <!-- Junta conectando o body ao base_link -->
+  <xacro:joint_fixed parent="base_link" child="body" z="${body_z_offset}"/>
+  <!-- Rodas e eixos -->
+  <xacro:wheels position="front"/>
+  <xacro:wheels position="rear"/>
   <!-- Juntas conectando os eixos ao body -->
-  <xacro:joint_fixed parent="body" child="wheel_front_axle" x="${0.5 * wheelbase}" z="${wheel_axle_z_offset}"/>
-  <xacro:joint_fixed parent="body" child="wheel_rear_axle" x="${-0.5 * wheelbase}" z="${wheel_axle_z_offset}"/>
-  <!-- Link base para conectar o body -->
-  <link name="base_link"/>
-  <xacro:joint_fixed parent="base_link" child="body" z="${body_z_offset}"/>
+  <xacro:joint_fixed
+    parent="body"
+    child="wheel_front_axle"
+    x="${0.5 * wheelbase}"
+    z="${wheel_axle_z_offset}"
+  />
+  <xacro:joint_fixed
+    parent="body"
+    child="wheel_rear_axle"
+    x="${-0.5 * wheelbase}"
+    z="${wheel_axle_z_offset}"
+  />
 </robot>

File: urdf/rosbot3.xacro (robot description, xacro)
@@ -6,5 +6,4 @@
 <robot name="rosbot3"  xmlns:xacro="http://www.ros.org/wiki/xacro">
   <xacro:include filename="$(find rosbot3_description)/urdf/base.xacro"/>
-  <!-- Propriedades do suporte e lidar -->
   <!-- Alturas baseadas nas especificações: base=103mm, support=141mm, lidar=197mm -->
   <xacro:property name="base_top_z" value="${103 * M}"/>
@@ -13,4 +12,15 @@
   <xacro:property name="lidar_height" value="${lidar_top_z - base_top_z}"/>
   <xacro:property name="lidar_size" value="${50 * M}"/>
+  <xacro:property name="lidar_offset_x" value="${30 * M}"/>
+  <!-- Dimensões do suporte da camera -->
+  <xacro:property name="camera_support_height" value="${94 * M}"/>
+  <xacro:property name="camera_support_size" value="${20 * M}"/>
+  <xacro:property name="camera_offset_x" value="${-30 * M}"/>
+  <xacro:solid_block
+    name="camera_support"
+    size_x="${camera_support_size}"
+    size_y="${camera_support_size}"
+    size_z="${camera_support_height}"
+  />
   <!-- Lidar -->
   <xacro:solid_block
@@ -21,10 +31,18 @@
   <!-- Link do laser (para o sensor LiDAR) -->
   <link name="laser"/>
-  <!-- Junta conectando o lidar ao body (posicionado no topo dos postes) -->
+  <!-- Junta conectando o lidar ao body (centrado no topo) -->
   <xacro:property name="lidar_z_joint" value="${0.5 * body_height + 0.5 * lidar_height}"/>
   <xacro:joint_fixed
     parent="body"
     child="lidar"
+    x="${lidar_offset_x}"
     z="${lidar_z_joint}"/>
+  <!-- Junta conectando o camera_support ao body (atrás do lidar) -->
+  <xacro:property name="camera_support_z_joint" value="${0.5 * body_height + 0.5 * camera_support_height}"/>
+  <xacro:joint_fixed
+    parent="body"
+    child="camera_support"
+    x="${camera_offset_x}"
+    z="${camera_support_z_joint}"/>
   <!-- Junta conectando o link laser ao lidar -->
   <xacro:joint_fixed
