Commit message: modelagem inicial base rodas e inicio do lidar

File: urdf/rosbot3.xacro (robot description, xacro)
@@ -1,48 +1,34 @@
 <?xml version="1.0" encoding="utf-8"?>
 <!--
-  Description of the ROSelito robot.
-  Author: Helio Perroni Filho
+  Description of the ROSbot3 robot.
+  Author: Gabryel Batista
 -->
-<robot name="rosbot3" xmlns:xacro="http://www.ros.org/wiki/xacro">
-  <xacro:include filename="$(find rosbot3_description)/urdf/ugv02.xacro"/>
-  <xacro:property name="payload_base_length" value="${156.22 * M}"/>
-  <xacro:property name="payload_base_width" value="${159.96 * M}"/>
-  <xacro:property name="payload_base_height" value="${42.7 * M}"/>
-  <xacro:property name="lidar_side" value="${45.61 * M}"/>
-  <xacro:property name="lidar_height" value="${37.6 * M}"/>
+<robot name="rosbot3"  xmlns:xacro="http://www.ros.org/wiki/xacro">
+  <xacro:include filename="$(find rosbot3_description)/urdf/base.xacro"/>
+  <!-- Propriedades do suporte e lidar -->
+  <!-- Alturas baseadas nas especificações: base=103mm, support=141mm, lidar=197mm -->
+  <xacro:property name="base_top_z" value="${103 * M}"/>
+  <xacro:property name="lidar_top_z" value="${141 * M}"/>
+  <!-- Dimensões do lidar -->
+  <xacro:property name="lidar_height" value="${lidar_top_z - base_top_z}"/>
+  <xacro:property name="lidar_size" value="${50 * M}"/>
+  <!-- Lidar -->
   <xacro:solid_block
-    name="payload_base"
-    size_x="${payload_base_length}"
-    size_y="${payload_base_width}"
-    size_z="${payload_base_height}"
-  />
+    name="lidar"
+    size_x="${lidar_size}"
+    size_y="${lidar_size}"
+    size_z="${lidar_height}"/>
+  <!-- Link do laser (para o sensor LiDAR) -->
+  <link name="laser"/>
+  <!-- Junta conectando o lidar ao body (posicionado no topo dos postes) -->
+  <xacro:property name="lidar_z_joint" value="${0.5 * body_height + 0.5 * lidar_height}"/>
   <xacro:joint_fixed
     parent="body"
-    child="payload_base"
-    z="${0.5 * (body_height + payload_base_height)}"
-  />
-  <xacro:camera_link name="camera_front"/>
-  <xacro:joint_fixed
-    parent="payload_base"
-    child="camera_front"
-    x="${0.5 * payload_base_length}"
-  />
-  <xacro:solid_block
-    name="lidar"
-    size_x="${lidar_side}"
-    size_y="${lidar_side}"
-    size_z="${lidar_height}"
-  />
-  <xacro:joint_fixed
-    parent="payload_base"
     child="lidar"
-    x="${0.5 * payload_base_height}"
-    z="${0.5 * (payload_base_height + lidar_height)}"
-  />
-  <link name="laser"/>
+    z="${lidar_z_joint}"/>
+  <!-- Junta conectando o link laser ao lidar -->
   <xacro:joint_fixed
     parent="lidar"
     child="laser"
-    z="${0.5 * lidar_height}"
-  />
+    z="${0.5 * lidar_height}"/>
 </robot>

Commit message: [1.0.0] Atualização do arquivo rosbot3.xacro com novas propriedades para a câmera e ajustes nas juntas

File: urdf/rosbot3.xacro (robot description, xacro)
@@ -6,5 +6,5 @@
 <robot name="rosbot3"  xmlns:xacro="http://www.ros.org/wiki/xacro">
   <xacro:include filename="$(find rosbot3_description)/urdf/base.xacro"/>
-  <!-- Alturas baseadas nas especificações: base=103mm, support=141mm, lidar=197mm -->
+  <!-- Alturas baseadas nas especificações disponíveis em https://husarion.com/manuals/rosbot/ -->
   <xacro:property name="base_top_z" value="${103 * M}"/>
   <xacro:property name="lidar_top_z" value="${141 * M}"/>
@@ -17,4 +17,8 @@
   <xacro:property name="camera_support_size" value="${20 * M}"/>
   <xacro:property name="camera_offset_x" value="${-30 * M}"/>
+  <!-- Dimensões da camera disponíveis em: https://shop.luxonis.com/products/oak-d-lite-1?variant=42583102456031 -->
+  <xacro:property name="camera_height" value="${28 * M}"/>
+  <xacro:property name="camera_width" value="${91 * M}"/>
+  <xacro:property name="camera_length" value="${17.5 * M}"/>
   <xacro:solid_block
     name="camera_support"
@@ -22,4 +26,16 @@
     size_y="${camera_support_size}"
     size_z="${camera_support_height}"
+  />
+  <xacro:solid_block
+    name="camera_block"
+    size_x="${camera_length}"
+    size_y="${camera_width}"
+    size_z="${camera_height}"
+  />
+  <xacro:camera_link name="camera_front"/>
+  <xacro:joint_fixed
+    parent="camera_support"
+    child="camera_front"
+    z="${camera_support_height}"
   />
   <!-- Lidar -->
@@ -31,5 +47,5 @@
   <!-- Link do laser (para o sensor LiDAR) -->
   <link name="laser"/>
-  <!-- Junta conectando o lidar ao body (centrado no topo) -->
+  <!-- Junta conectando o lidar ao body -->
   <xacro:property name="lidar_z_joint" value="${0.5 * body_height + 0.5 * lidar_height}"/>
   <xacro:joint_fixed
@@ -38,6 +54,11 @@
     x="${lidar_offset_x}"
     z="${lidar_z_joint}"/>
-  <!-- Junta conectando o camera_support ao body (atrás do lidar) -->
-  <xacro:property name="camera_support_z_joint" value="${0.5 * body_height + 0.5 * camera_support_height}"/>
+  <!-- Junta conectando o link laser ao lidar -->
+  <xacro:joint_fixed
+    parent="lidar"
+    child="laser"
+    z="${0.5 * lidar_height}"/>
+  <!-- Juntas relacionadas a camera -->
+  <xacro:property name="camera_support_z_joint" value="${base_top_z}"/>
   <xacro:joint_fixed
     parent="body"
@@ -45,8 +66,14 @@
     x="${camera_offset_x}"
     z="${camera_support_z_joint}"/>
-  <!-- Junta conectando o link laser ao lidar -->
   <xacro:joint_fixed
-    parent="lidar"
-    child="laser"
-    z="${0.5 * lidar_height}"/>
+    parent="camera_support"
+    child="camera_block"
+    x="${camera_length}"
+    z="${0.5* camera_support_height}"
+  />
+  <xacro:joint_fixed
+    parent="camera_block"
+    child="camera_front"
+    z="${0.5* camera_support_height}"
+  />
 </robot>

Commit message: [1.0.1] Adicionado braço horizontal para camera

File: urdf/rosbot3.xacro (robot description, xacro)
@@ -17,4 +17,8 @@
   <xacro:property name="camera_support_size" value="${20 * M}"/>
   <xacro:property name="camera_offset_x" value="${-30 * M}"/>
+  <!-- Dimensões do braço horizontal da camera -->
+  <xacro:property name="camera_arm_length" value="${60 * M}"/>
+  <xacro:property name="camera_arm_width" value="${15 * M}"/>
+  <xacro:property name="camera_arm_height" value="${15 * M}"/>
   <!-- Dimensões da camera disponíveis em: https://shop.luxonis.com/products/oak-d-lite-1?variant=42583102456031 -->
   <xacro:property name="camera_height" value="${28 * M}"/>
@@ -28,4 +32,10 @@
   />
   <xacro:solid_block
+    name="camera_arm"
+    size_x="${camera_arm_length}"
+    size_y="${camera_arm_width}"
+    size_z="${camera_arm_height}"
+  />
+  <xacro:solid_block
     name="camera_block"
     size_x="${camera_length}"
@@ -34,9 +44,4 @@
   />
   <xacro:camera_link name="camera_front"/>
-  <xacro:joint_fixed
-    parent="camera_support"
-    child="camera_front"
-    z="${camera_support_height}"
-  />
   <!-- Lidar -->
   <xacro:solid_block
@@ -65,15 +70,27 @@
     child="camera_support"
     x="${camera_offset_x}"
-    z="${camera_support_z_joint}"/>
+    z="${0.5 *camera_support_z_joint + 0.5 * camera_support_height - ground_clearance}"/>
+  <!-- Braço horizontal conectado ao topo do suporte vertical, apontando para frente -->
   <xacro:joint_fixed
     parent="camera_support"
+    child="camera_arm"
+    x="${0.5 * camera_arm_length}"
+    z="${0.5 * camera_support_height}"
+  />
+  <!-- Bloco da camera conectado ao final do braço horizontal -->
+  <!-- O final do braço está em x = 0.5 * camera_arm_length (do centro do braço) -->
+  <!-- O centro do bloco da camera precisa estar em x = 0.5 * camera_arm_length + 0.5 * camera_length -->
+  <xacro:joint_fixed
+    parent="camera_arm"
     child="camera_block"
-    x="${camera_length}"
-    z="${0.5* camera_support_height}"
+    x="${0.5 * camera_arm_length + 0.5 * camera_length}"
+    z="${0.5 * camera_arm_height}"
   />
+  <!-- Link da camera conectado ao bloco da camera -->
   <xacro:joint_fixed
     parent="camera_block"
     child="camera_front"
-    z="${0.5* camera_support_height}"
+    x="${0.5 * camera_length}"
+    z="${0.5 * camera_height}"
   />
 </robot>
